File: eagle/hackeeg-shield.brd (EAGLE design)
At the start: 101.6 x 53.3 mm, 146 parts, among them IC1 ADS1299IPAG, IC10 TXB0108PWR, IC11 TXB0108PWR, IC2 TPS72325DBVT, IC3 TPS73225DBVT, IC5 24AA256UID, IC6 TPS60403DBVT, IC7 OPA376DBV, IC8 OPA376DBV, IC9 TXS0102DCUR

Commit message: update to eagle 7.6
Parts:
- C65: value 1 uF -> 1uF
Changed lines of the file:
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@@
 <?xml version="1.0" encoding="utf-8"?>
 <!DOCTYPE eagle SYSTEM "eagle.dtd">
-<eagle version="6.5.0">
+<eagle version="7.6.0">
 <drawing>
 <settings>
@@
 <pass name="Default">
 <param name="RoutingGrid" value="10mil"/>
+<param name="AutoGrid" value="1"/>
+<param name="Efforts" value="0"/>
+<param name="TopRouterVariant" value="1"/>
 <param name="tpViaShape" value="round"/>
 <param name="PrefDir.1" value="|"/>
@@
 <attribute name="VALUE" x="53.7972" y="39.8272" size="0.4064" layer="27" font="vector" rot="R270"/>
 </element>
-<element name="C65" library="SparkFun-Passives" package="0603-CAP" value="1 uF" x="57.658" y="38.8112" smashed="yes" rot="R270">
+<element name="C65" library="SparkFun-Passives" package="0603-CAP" value="1uF" x="57.658" y="38.8112" smashed="yes" rot="R270">
 <attribute name="NAME" x="58.4708" y="39.878" size="0.762" layer="25" font="vector" ratio="12" rot="R270"/>
 <attribute name="VALUE" x="56.515" y="39.8272" size="0.4064" layer="27" font="vector" rot="R270"/>
